File: Electrical/circuitPNP/circuitPNP.kicad_pcb (KiCad board)
At the start: 2 copper layers, 87 parts, among them J1 USB_C_Receptacle_USB2.0_16P, J2 Screw_Terminal_01x02, J21 Conn_01x04_Pin, J22 Conn_01x04_Pin, J23 Conn_01x04_Pin, J24 Conn_01x04_Pin, J25 Conn_01x04_Pin, J26 Conn_01x02_Pin, J27 Conn_01x02_Pin, J28 Conn_01x04_Pin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

Commit message: pcb wip
Parts:
- added C22: 10uf, Capacitor_SMD:C_0603_1608Metric_Pad1.08x0.95mm_HandSolder, F.Cu at (112.5, 69.3)
- added C23: 0.1uf, Capacitor_SMD:C_0603_1608Metric_Pad1.08x0.95mm_HandSolder, F.Cu at (112.3, 73.6)
- added D2: D, Diode_SMD:D_SMB, F.Cu at (129.9, 98.2)
- added D4: D, Diode_SMD:D_SMB, F.Cu at (138.8, 98.1)
- added H1: MountingHole, MountingHole:MountingHole_3.2mm_M3, F.Cu at (200.9, 61.2)
- added H2: MountingHole, MountingHole:MountingHole_3.2mm_M3, F.Cu at (101.3, 61.0)
- added H3: MountingHole, MountingHole:MountingHole_3.2mm_M3, F.Cu at (200.8, 140.4)
- added H4: MountingHole, MountingHole:MountingHole_3.2mm_M3, F.Cu at (101.5, 140.6)
- C11, C15, C19, C20, C4, C6: value 100uF? -> 100uF
- J4: value Conn_01x04_Pin -> Conn_01x03_Pin; footprint Connector_PinSocket_2.54mm:PinSocket_1x04_P2.54mm_Vertical -> Connector_PinHeader_2.54mm:PinHeader_1x03_P2.54mm_Vertical
- moved R1 129.3 mm to (266.1, 45.9)
- moved C21 129.3 mm to (266.1, 43.4)
- moved C5 129.3 mm to (261.8, 43.4)
- moved C7 129.3 mm to (261.8, 45.9)
- moved R11 129.3 mm to (270.5, 43.4)
- moved R12 129.3 mm to (270.5, 45.9)
- moved R22 129.3 mm to (274.8, 43.4)
- moved R23 129.3 mm to (274.8, 45.9)
- moved C17 125.3 mm to (256.7, 32.3)
- moved C18 125.3 mm to (256.7, 34.8)
- moved C2 125.3 mm to (252.3, 32.3)
- moved R20 125.3 mm to (265.4, 32.3)
- moved R9 125.3 mm to (261.0, 32.3)
- moved C3 125.3 mm to (252.3, 34.8)
- moved R10 125.3 mm to (261.0, 34.8)
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Connections:
- A2 pad 9: /GPIO13 -> /GPIO46
- J4 pad 1: /3V3 -> /TX
- J4 pad 2: /TX -> /RX
- J4 pad 3: /RX -> GND
- J6 pad 1: /CANH -> GND
- J6 pad 3: GND -> /CANH
- R22 pad 1: /GPIO13 -> /GPIO3
- SW3 pad 1: /5V_BUCK -> /VBus
- SW3 pad 3: /VBus -> /5V_BUCK
Routing:
- added copper zone on In1.Cu, net /24V
- added copper zone on In1.Cu, net /3V3
- added copper zone on In2.Cu, net GND
Other:
- board outline added: 109.2 x 91.6 mm
- copper layers 2 -> 4

Commit message: wip pcb
Parts:
- J2, J3: footprint TerminalBlock:TerminalBlock_MaiXu_MX126-5.0-02P_1x02_P5.00mm -> Connector_Molex:Molex_KK-396_A-41792-0002_1x02_P3.96mm_Horizontal
- J22, J23, J24, J25: footprint Connector_Molex:Molex_KK-254_AE-6410-04A_1x04_P2.54mm_Vertical -> Connector_Molex:Molex_KK-396_A-41792-0004_1x04_P3.96mm_Horizontal
- moved R11 172.8 mm to (113.7, 116.1), turned to -90 degrees
- moved R9 171.7 mm to (111.2, 116.1), turned to -90 degrees
- moved C5 163.1 mm to (126.6, 134.6)
- moved C21 157.8 mm to (121.1, 105.6), turned to 90 degrees
- moved R2 157.3 mm to (108.0, 89.5)
- moved R3 156.7 mm to (108.0, 87.9)
- moved C2 154.9 mm to (104.0, 76.9)
- moved C1 149.3 mm to (99.9, 76.9)
- moved R13 143.7 mm to (134.1, 116.1), turned to -90 degrees
- moved C3 143.6 mm to (149.4, 135.0)
- moved R14 140.4 mm to (136.7, 116.1), turned to -90 degrees
- moved R5 138.4 mm to (104.0, 81.2)
- moved C8 138.2 mm to (122.4, 86.1)
- moved R22 136.8 mm to (141.9, 75.6)
- moved C18 135.8 mm to (128.4, 79.5)
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Connections:
- R1 pad 2: GND -> /3V3
Routing:
- net GND: track 0.00 -> 60.4 mm, vias 0 -> 24
- net /24V: track 0.00 -> 59.7 mm, vias 0 -> 9
- net /GPIO35: track 0.00 -> 48.3 mm, vias 0 -> 2
- net /3V3: track 0.00 -> 48.3 mm, vias 0 -> 21
- net /GPIO36: track 0.00 -> 42.5 mm, vias 0 -> 2
- net /GPIO37: track 0.00 -> 37.0 mm, vias 0 -> 2
- net /CANH: track 0.00 -> 23.5 mm
- net /CANL: track 0.00 -> 22.7 mm
- net /GPIO2: track 0.00 -> 20.0 mm
- net /GPIO1: track 0.00 -> 18.3 mm
- net /GPIO0: track 0.00 -> 15.7 mm
- net /VBus: track 0.00 -> 8.67 mm
- net Net-(J1-D+-PadA6): track 0.00 -> 5.03 mm
- net /GPIO48: track 0.00 -> 5.02 mm
- net /GPIO47: track 0.00 -> 4.92 mm
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Other:
- board size 109.2 x 91.6 mm -> 109.2 x 104.7 mm

Commit message: pcb done, wainting for circuit testing
Parts:
- added D5: LED, LED_SMD:LED_0603_1608Metric, F.Cu at (182.6, 79.0)
- added D6: LED, LED_SMD:LED_0603_1608Metric, F.Cu at (101.1, 77.2)
- added G***: LOGO, LOGO, F.Cu at (140.1, 103.9)
- added G***: LOGO, LOGO, F.Cu at (163.3, 103.8)
- added R36: 330, Resistor_SMD:R_0603_1608Metric_Pad0.98x0.95mm_HandSolder, F.Cu at (179.4, 79.0)
- added R37: 330, Resistor_SMD:R_0603_1608Metric_Pad0.98x0.95mm_HandSolder, F.Cu at (104.9, 77.2)
- added TP1: TestPoint, TestPoint:TestPoint_Pad_D2.0mm, F.Cu at (106.2, 113.5)
- added TP2: TestPoint, TestPoint:TestPoint_Pad_D2.0mm, F.Cu at (109.3, 70.9)
- added TP3: TestPoint, TestPoint:TestPoint_Pad_D2.0mm, F.Cu at (118.3, 71.0)
- added TP4: TestPoint, TestPoint:TestPoint_Pad_D2.0mm, F.Cu at (195.5, 70.3)
- added TP5: TestPoint, TestPoint:TestPoint_Pad_D2.0mm, F.Cu at (157.0, 59.5)
- added TP6: TestPoint, TestPoint:TestPoint_Pad_D2.0mm, F.Cu at (105.8, 99.5)
- added TP7: TestPoint, TestPoint:TestPoint_Pad_D2.0mm, F.Cu at (152.0, 59.5)
- added TP8: TestPoint, TestPoint:TestPoint_Pad_D2.0mm, F.Cu at (119.8, 86.8)
- DRIVE X: renamed from A4
- DRIVE Y: renamed from A3
- DRIVE YAW: renamed from A1
- DRIVE Z: renamed from A2
- moved J21 37.8 mm to (201.9, 98.9), turned to 90 degrees
- moved R18 23.1 mm to (194.1, 91.1), turned to 180 degrees
- moved R17 22.8 mm to (194.2, 93.8), turned to 180 degrees
- moved C1 19.8 mm to (110.2, 93.8), turned to 90 degrees
- moved C2 19.1 mm to (112.9, 93.8), turned to 90 degrees
- moved C17 11.3 mm to (169.1, 58.5), turned to -90 degrees
- moved D7 7.43 mm to (193.7, 84.4), turned to 0 degrees
- moved SW2 6.68 mm to (164.7, 63.0), turned to 180 degrees
- moved J8 6.50 mm to (201.8, 105.0)
- moved R21 6.40 mm to (196.7, 105.1)
- moved C16 6.18 mm to (166.4, 58.5), turned to -90 degrees
- moved R20 6.07 mm to (196.6, 111.5)
- moved J7 5.92 mm to (201.8, 111.4)
- moved J5 5.49 mm to (201.8, 117.6)
- moved R19 5.41 mm to (196.6, 117.8)
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Connections:
- D2 pad 1: /5V -> /5V_BUCK
- D4 pad 1: /5V -> /5V_BUCK
- DRIVE X pad 15: /GPIO15 -> /GPIO7
- DRIVE X pad 16: /GPIO7 -> /GPIO6
- DRIVE X pad 9: /GPIO16 -> /GPIO15
- DRIVE Y pad 15: /GPIO18 -> /GPIO17
- DRIVE Y pad 16: /GPIO17 -> /GPIO16
- DRIVE Y pad 9: /GPIO10 -> /GPIO18
- DRIVE YAW pad 15: /GPIO5 -> /GPIO13
- DRIVE YAW pad 16: /GPIO4 -> /GPIO12
- DRIVE YAW pad 9: /GPIO6 -> /GPIO14
- DRIVE Z pad 15: /GPIO12 -> /GPIO46
- DRIVE Z pad 16: /GPIO11 -> /GPIO3
- DRIVE Z pad 9: /GPIO46 -> /GPIO11
- J26 pad 1: /5V -> /5V_BUCK
- J27 pad 1: /5V -> /5V_BUCK
- R22 pad 1: /GPIO3 -> /GPIO5
- R23 pad 1: /GPIO21 -> /GPIO4
- SW3 pad 4: GND -> unconnected-(SW3-A-Pad4)
- SW3 pad 5: GND -> unconnected-(SW3-B-Pad5)
- SW3 pad 6: GND -> unconnected-(SW3-C-Pad6)
Routing:
- net /3V3: track 48.3 -> 253.6 mm, vias 21 -> 18
- net /GPIO6: track 0.00 -> 91.7 mm, vias 0 -> 1
- net /GPIO7: track 0.00 -> 89.6 mm, vias 0 -> 1
- net /GPIO15: track 0.00 -> 76.8 mm, vias 0 -> 1
- net /GPIO16: track 0.00 -> 73.5 mm, vias 0 -> 1
- net /GPIO17: track 0.00 -> 71.2 mm, vias 0 -> 1
- net /5V_BUCK: track 0.00 -> 70.5 mm
- net /D-: track 1.93 -> 71.2 mm
- net /D+: track 1.99 -> 71.1 mm
- net /GPIO18: track 0.00 -> 63.7 mm, vias 0 -> 1
- net /GPIO3: track 0.00 -> 57.7 mm, vias 0 -> 1
- net /GPIO46: track 0.00 -> 56.6 mm, vias 0 -> 1
- net /GPIO11: track 0.00 -> 49.2 mm, vias 0 -> 1
- net /GPIO14: track 0.00 -> 48.8 mm, vias 0 -> 1
- net /GPIO12: track 0.00 -> 47.2 mm, vias 0 -> 1
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- added copper zone on B.Cu, net GND
- added copper zone on F.Cu, net GND
Other:
- board size 109.2 x 104.7 mm -> 109.2 x 104.6 mm
- board text added: "+"
- board text added: "24V"
- board text added: "3V3"
- board text added: "5V"
- board text added: "5V_BUCK"
- board text added: "5V_USB"
- board text added: "AIR PUMP"
- board text added: "CAN"
- board text added: "G"
- board text added: "GND"
- board text added: "H"
- board text added: "L"
- board text added: "Limit switchs"
- board text added: "M2 M1 M0"
- board text added: "PickUS & PlacUS"
- board text added: "Pressure"
- board text added: "RX"
- board text added: "SCL"
- board text added: "SDA"
- board text added: "Solenoid"
- board text added: "TX"

Commit message: missed that
Routing:
- added copper zone on In2.Cu, net /24V
- added copper zone on In2.Cu, net /3V3
- added copper zone on In1.Cu, net GND
- removed copper zone on In1.Cu, net /24V
- removed copper zone on In1.Cu, net /3V3
- removed copper zone on In2.Cu, net GND
Changed lines of the file:
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@@
 	(layers
 		(0 "F.Cu" signal)
-		(4 "In1.Cu" signal "VCC")
-		(6 "In2.Cu" signal "GND")
+		(4 "In1.Cu" signal "GND")
+		(6 "In2.Cu" signal "VCC")
 		(2 "B.Cu" signal)
 		(9 "F.Adhes" user "F.Adhesive")
@@
 			(outputformat 1)
 			(mirror no)
-			(drillshape 1)
+			(drillshape 0)
 			(scaleselection 1)
 			(outputdirectory "")
@@
 		(min_thickness 0.25)
 		(filled_areas_thickness no)
-		(fill
+		(fill yes
 			(thermal_gap 0.5)
 			(thermal_bridge_width 0.5)
@@
 		(min_thickness 0.25)
 		(filled_areas_thickness no)
-		(fill
+		(fill yes
 			(thermal_gap 0.5)
 			(thermal_bridge_width 0.5)
@@
 	)
 	(zone
-		(net 57)
-		(net_name "/3V3")
+		(net 11)
+		(net_name "GND")
 		(layer "In1.Cu")
 		(hatch edge 0.5)
@@
 		(min_thickness 0.25)
 		(filled_areas_thickness no)
-		(fill
+		(fill yes
 			(thermal_gap 0.5)
 			(thermal_bridge_width 0.5)
@@
 		(polygon
 			(pts
-				(xy 96.52 55.88) (xy 96.656913 99.044002) (xy 205.74 99.06) (xy 205.74 55.88)
+				(xy 96.52 55.88) (xy 205.864 55.734) (xy 205.864 160.563) (xy 96.52 160.598)
 			)
 		)
@@
 		(net 7)
 		(net_name "/24V")
-		(layer "In1.Cu")
+		(layer "In2.Cu")
 		(hatch edge 0.5)
-		(priority 1)
 		(connect_pads
 			(clearance 0.5)
@@
 		(min_thickness 0.25)
 		(filled_areas_thickness no)
-		(fill
+		(fill yes
 			(thermal_gap 0.5)
 			(thermal_bridge_width 0.5)
@@
 		(polygon
 			(pts
-				(xy 96.515533 160.563) (xy 96.9659 105.8322) (xy 205.74 105.8322) (xy 205.74 160.563)
+				(xy 205.74 160.563) (xy 96.52 160.598) (xy 96.7846 106.2736) (xy 205.74 106.68)
 			)
 		)
 	)
 	(zone
-		(net 11)
-		(net_name "GND")
+		(net 57)
+		(net_name "/3V3")
 		(layer "In2.Cu")
 		(hatch edge 0.5)
+		(priority 1)
 		(connect_pads
 			(clearance 0.5)
@@
 		(min_thickness 0.25)
 		(filled_areas_thickness no)
-		(fill
+		(fill yes
 			(thermal_gap 0.5)
 			(thermal_bridge_width 0.5)
@@
 		(polygon
 			(pts
-				(xy 96.52 55.88) (xy 96.52 160.598) (xy 205.74 160.598) (xy 205.74 55.88)
+				(xy 96.52 55.88) (xy 96.52 97.79) (xy 205.74 98.425) (xy 205.864 55.734)
 			)
 		)

Commit message: pull down on gate for mosfet
Parts:
- removed Q2: IRLML6344TRPBF, Package_TO_SOT_SMD:SOT-23
- added Q3: IRLML6244, Package_TO_SOT_SMD:SOT-23, F.Cu at (140.5, 71.1)
- added R38: 10k 1%, Resistor_SMD:R_0603_1608Metric_Pad0.98x0.95mm_HandSolder, F.Cu at (139.4, 74.9)
- added R39: 10k 1%, Resistor_SMD:R_0603_1608Metric_Pad0.98x0.95mm_HandSolder, F.Cu at (147.4, 74.7)
- A1: renamed from DRIVE YAW
- A2: renamed from DRIVE Z
- A3: renamed from DRIVE Y
- A4: renamed from DRIVE X
- Q1: value IRLML6344TRPBF -> IRLML6244
- moved Q1 7.85 mm to (148.5, 70.9)
- moved R22 0.10 mm to (141.5, 74.9)
Connections:
- Q1 pad 1: GND -> Net-(Q1-G)
- Q1 pad 2: Net-(Q1-G) -> GND
- Q1 pad 3: Net-(D2-A) -> Net-(D4-A)
- R22 pad 2: Net-(Q1-G) -> Net-(Q3-G)
- R23 pad 2: Net-(Q2-G) -> Net-(Q1-G)
Routing:
- net Net-(Q3-G): track 0.00 -> 4.08 mm
- net Net-(Q2-G): track 1.88 -> 0.00 mm
- net Net-(Q1-G): track 2.02 -> 3.87 mm
- net /CANL: track 17.4 -> 16.9 mm
- net /24V: track 65.2 -> 65.0 mm, vias 9 -> 8

Commit message: fabricationFile for v1
Parts:
- R38, R39: value 10k 1% -> 10k
- moved Q3 7.98 mm to (148.5, 71.0)
- moved Q1 7.93 mm to (140.6, 70.9)
- moved R39 0.15 mm to (147.6, 74.7)
- moved R38 0.15 mm to (139.6, 74.9)
Connections:
- J22 pad 3: Net-(A1-A2) -> Net-(A1-A1)
- J22 pad 4: Net-(A1-A1) -> Net-(A1-A2)
- J23 pad 3: Net-(A4-A2) -> Net-(A4-A1)
- J23 pad 4: Net-(A4-A1) -> Net-(A4-A2)
- J24 pad 3: Net-(A3-A2) -> Net-(A3-A1)
- J24 pad 4: Net-(A3-A1) -> Net-(A3-A2)
- J25 pad 3: Net-(A2-A2) -> Net-(A2-A1)
- J25 pad 4: Net-(A2-A1) -> Net-(A2-A2)
- Q1 pad 3: Net-(D4-A) -> Net-(D2-A)
- Q3 pad 3: Net-(D2-A) -> Net-(D4-A)
- R22 pad 2: Net-(Q3-G) -> Net-(Q1-G)
- R23 pad 2: Net-(Q1-G) -> Net-(Q3-G)
- R38 pad 1: Net-(Q3-G) -> Net-(Q1-G)
- R39 pad 1: Net-(Q1-G) -> Net-(Q3-G)
Routing:
- net Net-(A4-A1): track 19.2 -> 17.5 mm
- net Net-(A2-A1): track 18.9 -> 17.3 mm
- net Net-(A1-A1): track 18.8 -> 17.2 mm
- net Net-(A3-A1): track 18.9 -> 17.2 mm
- net /GPIO5: track 37.7 -> 38.7 mm
- net Net-(A4-A2): track 17.1 -> 18.1 mm
- net Net-(A2-A2): track 17.1 -> 17.8 mm
- net Net-(A3-A2): track 17.3 -> 17.8 mm
