File: Electrical/circuitPNP/circuitPNP.kicad_sch (KiCad schematic)
At the start: 105 parts, among them J1 USB_C_Receptacle_USB2.0_16P, J2 Screw_Terminal_01x02, J21 Conn_01x04_Pin, J22 Conn_01x04_Pin, J23 Conn_01x04_Pin, J24 Conn_01x04_Pin, J25 Conn_01x04_Pin, J26 Conn_01x02_Pin, J27 Conn_01x02_Pin, J28 Conn_01x04_Pin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

Commit message: fabricationFile for v1
Parts:
- removed Q1, Q2: IRLML6344TRPBF, Package_TO_SOT_SMD:SOT-23, symbol Transistor_FET:GS66504B
- added Q1, Q3: IRLML6244, Package_TO_SOT_SMD:SOT-23, symbol Transistor_FET:IRLML6244
- added R38, R39: 10k, Resistor_SMD:R_0603_1608Metric_Pad0.98x0.95mm_HandSolder, symbol Device:R
Connections:
- net GND: now also Q1.2 (S), Q3.2 (S), R38.2, R39.2
- net at A1.3 (A2): now also J22.4 (Pin_4); no longer J22.3 (Pin_3)
- net at A1.4 (A1): now also J22.3 (Pin_3); no longer J22.4 (Pin_4)
- net at A4.3 (A2): now also J23.4 (Pin_4); no longer J23.3 (Pin_3)
- net at A4.4 (A1): now also J23.3 (Pin_3); no longer J23.4 (Pin_4)
- net at A3.3 (A2): now also J24.4 (Pin_4); no longer J24.3 (Pin_3)
- net at A3.4 (A1): now also J24.3 (Pin_3); no longer J24.4 (Pin_4)
- net at R23.2: now also Q3.1 (G), R39.1
- net at D4.2 (A), J27.2 (Pin_2): now also Q3.3 (D)
- net at A2.3 (A2): now also J25.4 (Pin_4); no longer J25.3 (Pin_3)
- net at A2.4 (A1): now also J25.3 (Pin_3); no longer J25.4 (Pin_4)
- net at R22.2: now also Q1.1 (G), R38.1
- net at D2.2 (A), J26.2 (Pin_2): now also Q1.3 (D)
Other:
- moved on the sheet: R22, R23
